File: KiCad Projects/MIG Dumper/MIG Dumper.kicad_pcb (KiCad board)
At the start: 4 copper layers, 60 x 33 mm, 73 parts, among them J1 USB_C_Receptacle_USB2.0_16P, J2 Conn_02x04_Counter_Clockwise, J3 Conn_01x17_MountingPin, U1 ESP32-S2, U2 ICE40UP5K-SG48ITR, U3 GL823K-HCY04, U4 MAX20022ATIA+, Y1 ECS-400-10-37B2-CKY-TR

Commit message: Updated Flashcart PCB, uploaded Flashcart BOM
Revised the Flashcart PCB to the newer revision of the MIG v2, as well as added DigiKey and Mouser BOMs for the Flashcart. One capacitor measurement on the Dumper PCB was corrected as well.
Parts:
- C15: value 1u -> 110n
Connections:
- net CMD renamed IOB_4a
Changed lines of the file:
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@@
 	(net 7 "unconnected-(J2-Pin_3-Pad3)")
 	(net 8 "GPIO19")
-	(net 9 "CMD")
+	(net 9 "IOB_4a")
 	(net 10 "VDD")
 	(net 11 "GPIO7")
@@
 			(size 1.2 0.4)
 			(layers "F.Cu" "F.Paste" "F.Mask")
-			(net 9 "CMD")
+			(net 9 "IOB_4a")
 			(pinfunction "CMD")
 			(pintype "bidirectional")
@@
 			(layers "F.Cu" "F.Paste" "F.Mask")
 			(roundrect_rratio 0.25)
-			(net 9 "CMD")
+			(net 9 "IOB_4a")
 			(pinfunction "IOB_4a")
 			(pintype "bidirectional")
@@
 			)
 		)
-		(property "Value" "1u"
+		(property "Value" "110n"
 			(at 0 -1.43 90)
 			(layer "B.Fab")
