File: KiCad Projects/MIG Flashcart/Capacitors.kicad_sch (KiCad schematic)
At the start: 17 parts

Commit message: Updated Flashcart PCB, uploaded Flashcart BOM
Revised the Flashcart PCB to the newer revision of the MIG v2, as well as added DigiKey and Mouser BOMs for the Flashcart. One capacitor measurement on the Dumper PCB was corrected as well.
Parts:
- removed C5: C, Capacitor_SMD:C_0201_0603Metric, symbol Device:C
- C1, C11, C12, C20, C3, C8, C9: value C -> 0.82u
- C10, C15, C2: value C -> 0.88u
- C16: value 1u -> 0.88u
- C17, C18, C19: value 1u -> 0.82u
- C5: renamed from C6; value C -> 0.82u
- C6: renamed from C7; value C -> 3u3
Other:
- moved on the sheet: C10, C19, C2
