File: KiCad Projects/MIG Flashcart/MIG Flashcart.kicad_sch (KiCad schematic)
At the start: 18 parts, among them J1 Conn_02x04_Counter_Clockwise, J2 Conn_01x17, J3 1040310811, SW1 EVQ-P7A01P, U1 ICE40UP5K-SG48ITR, U2 ESP32-S2, U3 TLV70012_SOT353, U4 TLV70025_SOT353, Y1 ECS-400-10-37B2-CKY-TR

Commit message: Updated Flashcart PCB, uploaded Flashcart BOM
Revised the Flashcart PCB to the newer revision of the MIG v2, as well as added DigiKey and Mouser BOMs for the Flashcart. One capacitor measurement on the Dumper PCB was corrected as well.
Parts:
- added C7: DNP, Capacitor_SMD:C_0201_0603Metric, symbol Device:C
- added R1: 50R, Resistor_SMD:R_0201_0603Metric, symbol Device:R
- added TP1: TestPoint, MIG Flashcart:TestPoint_Pad_D0.5mm, symbol Connector:TestPoint
- C4: value C -> 0.82u
- renumbered R1 to R2, R2 to R4, R4 to R5, R5 to R6
Connections:
- net GND: now also U1.42 (IOT_51a), C7.2
- net IOB_3b: now also R1.1; no longer J3.5 (CLK)
- net at U2.48 (U0TXD): now also TP1.1
- new net: C7.1, J3.5 (CLK), R1.2
- no-connect marks 39 -> 37
